Commit message: Fix up mesh filepaths in kuka allegro and allegro urdf

File: assets/urdf/kuka_allegro_description/allegro_touch_sensor.urdf (robot description, URDF)
Before this commit: robot kuka_allegro, 22 links, 21 joints
Links:
- link allegro_mount: geometry collision mesh filename=meshes/mounts/allegro_mount.obj; visual mesh filename=meshes/mounts/allegro_mount.obj
- link index_link_0: geometry collision mesh filename=meshes/allegro/primary_base.obj; visual mesh filename=meshes/allegro/primary_base.obj
- link index_link_1: geometry collision mesh filename=meshes/allegro/primary_proximal.obj; visual mesh filename=meshes/allegro/primary_proximal.obj
- link index_link_2: geometry collision mesh filename=meshes/allegro/primary_medial.obj; visual mesh filename=meshes/allegro/primary_medial.obj
- link middle_link_0: geometry collision mesh filename=meshes/allegro/primary_base.obj; visual mesh filename=meshes/allegro/primary_base.obj
- link middle_link_1: geometry collision mesh filename=meshes/allegro/primary_proximal.obj; visual mesh filename=meshes/allegro/primary_proximal.obj
- link middle_link_2: geometry collision mesh filename=meshes/allegro/primary_medial.obj; visual mesh filename=meshes/allegro/primary_medial.obj
- link palm_link: geometry collision mesh filename=meshes/allegro/base_link.obj; visual mesh filename=meshes/allegro/base_link.obj
- link ring_link_0: geometry collision mesh filename=meshes/allegro/primary_base.obj; visual mesh filename=meshes/allegro/primary_base.obj
- link ring_link_1: geometry collision mesh filename=meshes/allegro/primary_proximal.obj; visual mesh filename=meshes/allegro/primary_proximal.obj
- link ring_link_2: geometry collision mesh filename=meshes/allegro/primary_medial.obj; visual mesh filename=meshes/allegro/primary_medial.obj
- link thumb_link_0: geometry collision mesh filename=meshes/allegro/thumb_base.obj; visual mesh filename=meshes/allegro/thumb_base.obj
- link thumb_link_1: geometry collision mesh filename=meshes/allegro/thumb_proximal.obj; visual mesh filename=meshes/allegro/thumb_proximal.obj
- link thumb_link_2: geometry collision mesh filename=meshes/allegro/thumb_medial.obj; visual mesh filename=meshes/allegro/thumb_medial.obj

File: assets/urdf/kuka_allegro_description/kuka_allegro_touch_sensor.urdf (robot description, URDF)
Before this commit: robot kuka_allegro, 28 links, 27 joints
Links:
- link allegro_mount: geometry collision mesh filename=meshes/mounts/allegro_mount.obj; visual mesh filename=meshes/mounts/allegro_mount.obj
- link iiwa7_link_0: geometry collision mesh filename=meshes/iiwa7/collision/link_0.obj; visual mesh filename=meshes/iiwa7/visual/link_0.obj
- link iiwa7_link_1: geometry collision mesh filename=meshes/iiwa7/collision/link_1.obj; visual mesh filename=meshes/iiwa7/visual/link_1.obj
- link iiwa7_link_2: geometry collision mesh filename=meshes/iiwa7/collision/link_2.obj; visual mesh filename=meshes/iiwa7/visual/link_2.obj
- link iiwa7_link_3: geometry collision mesh filename=meshes/iiwa7/collision/link_3.obj; visual mesh filename=meshes/iiwa7/visual/link_3.obj
- link iiwa7_link_4: geometry collision mesh filename=meshes/iiwa7/collision/link_4.obj; visual mesh filename=meshes/iiwa7/visual/link_4.obj
- link iiwa7_link_5: geometry collision mesh filename=meshes/iiwa7/collision/link_5.obj; visual mesh filename=meshes/iiwa7/visual/link_5.obj
- link iiwa7_link_6: geometry collision mesh filename=meshes/iiwa7/collision/link_6.obj; visual mesh filename=meshes/iiwa7/visual/link_6.obj
- link iiwa7_link_7: geometry collision mesh filename=meshes/iiwa7/collision/link_7.obj; visual mesh filename=meshes/iiwa7/visual/link_7.obj
- link index_link_0: geometry collision mesh filename=meshes/allegro/primary_base.obj; visual mesh filename=meshes/allegro/primary_base.obj
- link index_link_1: geometry collision mesh filename=meshes/allegro/primary_proximal.obj; visual mesh filename=meshes/allegro/primary_proximal.obj
- link index_link_2: geometry collision mesh filename=meshes/allegro/primary_medial.obj; visual mesh filename=meshes/allegro/primary_medial.obj
- link middle_link_0: geometry collision mesh filename=meshes/allegro/primary_base.obj; visual mesh filename=meshes/allegro/primary_base.obj
- link middle_link_1: geometry collision mesh filename=meshes/allegro/primary_proximal.obj; visual mesh filename=meshes/allegro/primary_proximal.obj
- link middle_link_2: geometry collision mesh filename=meshes/allegro/primary_medial.obj; visual mesh filename=meshes/allegro/primary_medial.obj
- link palm_link: geometry collision mesh filename=meshes/allegro/base_link.obj; visual mesh filename=meshes/allegro/base_link.obj
- link ring_link_0: geometry collision mesh filename=meshes/allegro/primary_base.obj; visual mesh filename=meshes/allegro/primary_base.obj
- link ring_link_1: geometry collision mesh filename=meshes/allegro/primary_proximal.obj; visual mesh filename=meshes/allegro/primary_proximal.obj
- link ring_link_2: geometry collision mesh filename=meshes/allegro/primary_medial.obj; visual mesh filename=meshes/allegro/primary_medial.obj
- link thumb_link_0: geometry collision mesh filename=meshes/allegro/thumb_base.obj; visual mesh filename=meshes/allegro/thumb_base.obj
- link thumb_link_1: geometry collision mesh filename=meshes/allegro/thumb_proximal.obj; visual mesh filename=meshes/allegro/thumb_proximal.obj
- link thumb_link_2: geometry collision mesh filename=meshes/allegro/thumb_medial.obj; visual mesh filename=meshes/allegro/thumb_medial.obj

Commit message: Hack fix to make viser allegro match allegro kuka

File: assets/urdf/kuka_allegro_description/allegro_touch_sensor.urdf (robot description, URDF)
Before this commit: robot allegro, 22 links, 21 joints
Links:
- removed link index_biotac_tip
- removed link middle_biotac_tip
- removed link ring_biotac_tip
- removed link thumb_biotac_tip
Joints:
- removed joint index_biotac_tip_joint
- removed joint middle_biotac_tip_joint
- removed joint ring_biotac_tip_joint
- removed joint thumb_biotac_tip_joint
- joint allegro_mount_joint: origin xyz=-0.008219 -0.02063 0.08086 rpy=0 -1.5708 0.785398 -> xyz=0.008219 -0.02063 0.08086 rpy=0 -1.5708 0.785398
