Commit message: Adjust hand mount to work

File: assets/urdf/kuka_allegro_description/iiwa14_sharpa.urdf (robot description, URDF)
Before this commit: robot kuka_allegro, 43 links, 42 joints
Joints:
- joint allegro_mount_joint: origin xyz=0.01 -0.02063 0.08 rpy=0 -1.5708 1.5708 -> xyz=0.0 0.0 0.04 rpy=0 0 -1.5708
