Commit message: Add left and right sharpa with iiwa

File: assets/urdf/kuka_allegro_description/iiwa14_left_sharpa.urdf (robot description, URDF)
Before this commit: robot kuka_allegro, 43 links, 42 joints
Links:
- removed link right_hand_C_MC
- removed link right_index_DP
- removed link right_index_MCP_VL
- removed link right_index_MP
- removed link right_index_PP
- removed link right_index_elastomer
- removed link right_index_fingertip
- removed link right_middle_DP
- removed link right_middle_MCP_VL
- removed link right_middle_MP
- removed link right_middle_PP
- removed link right_middle_elastomer
- removed link right_middle_fingertip
- removed link right_pinky_DP
- removed link right_pinky_MC
- removed link right_pinky_MCP_VL
- removed link right_pinky_MP
- removed link right_pinky_PP
- removed link right_pinky_elastomer
- removed link right_pinky_fingertip
- removed link right_ring_DP
- removed link right_ring_MCP_VL
- removed link right_ring_MP
- removed link right_ring_PP
- removed link right_ring_elastomer
- removed link right_ring_fingertip
- removed link right_thumb_CMC_VL
- removed link right_thumb_DP
- removed link right_thumb_MC
- removed link right_thumb_MCP_VL
- removed link right_thumb_PP
- removed link right_thumb_elastomer
- removed link right_thumb_fingertip
- added link left_hand_C_MC, mass 0.72045; collision mesh filename=left_sharpa_meshes/left_hand_C_MC.STL; visual mesh filename=left_sharpa_meshes/left_hand_C_MC_visual.STL
- added link left_index_DP, mass 0.003002; collision mesh filename=left_sharpa_meshes/left_DP.STL; visual mesh filename=left_sharpa_meshes/left_DP_visual.STL
- added link left_index_MCP_VL, mass 1.0E-06; collision mesh filename=left_sharpa_meshes/MCP_VL.STL; visual mesh filename=left_sharpa_meshes/left_MCP_VL_visual.STL
- added link left_index_MP, mass 0.02509; collision mesh filename=left_sharpa_meshes/left_MP.STL; visual mesh filename=left_sharpa_meshes/left_MP_visual.STL
- added link left_index_PP, mass 0.04138; collision mesh filename=left_sharpa_meshes/left_PP.STL; visual mesh filename=left_sharpa_meshes/left_PP_visual.STL
- added link left_index_elastomer, mass 0.00110; collision mesh filename=left_sharpa_meshes/elastomer.STL; visual mesh filename=left_sharpa_meshes/elastomer_surface.STL
- added link left_index_fingertip, mass 1.0E-06
- added link left_middle_DP, mass 0.003002; collision mesh filename=left_sharpa_meshes/left_DP.STL; visual mesh filename=left_sharpa_meshes/left_DP_visual.STL
- added link left_middle_MCP_VL, mass 1.0E-06; collision mesh filename=left_sharpa_meshes/MCP_VL.STL; visual mesh filename=left_sharpa_meshes/left_MCP_VL_visual.STL
- added link left_middle_MP, mass 0.02509; collision mesh filename=left_sharpa_meshes/left_MP.STL; visual mesh filename=left_sharpa_meshes/left_MP_visual.STL
- added link left_middle_PP, mass 0.04138; collision mesh filename=left_sharpa_meshes/left_PP.STL; visual mesh filename=left_sharpa_meshes/left_PP_visual.STL
- added link left_middle_elastomer, mass 0.00110; collision mesh filename=left_sharpa_meshes/elastomer.STL; visual mesh filename=left_sharpa_meshes/elastomer_surface.STL
- added link left_middle_fingertip, mass 1.0E-06
- added link left_pinky_DP, mass 0.003002; collision mesh filename=left_sharpa_meshes/left_DP.STL; visual mesh filename=left_sharpa_meshes/left_DP_visual.STL
- added link left_pinky_MC, mass 0.12541; collision mesh filename=left_sharpa_meshes/left_pinky_MC.STL; visual mesh filename=left_sharpa_meshes/left_pinky_MC_visual.STL
- added link left_pinky_MCP_VL, mass 1.0E-06; collision mesh filename=left_sharpa_meshes/MCP_VL.STL; visual mesh filename=left_sharpa_meshes/left_MCP_VL_visual.STL
- added link left_pinky_MP, mass 0.02509; collision mesh filename=left_sharpa_meshes/left_MP.STL; visual mesh filename=left_sharpa_meshes/left_MP_visual.STL
- added link left_pinky_PP, mass 0.04138; collision mesh filename=left_sharpa_meshes/left_PP.STL; visual mesh filename=left_sharpa_meshes/left_PP_visual.STL
- added link left_pinky_elastomer, mass 0.00110; collision mesh filename=left_sharpa_meshes/elastomer.STL; visual mesh filename=left_sharpa_meshes/elastomer_surface.STL
- added link left_pinky_fingertip, mass 1.0E-06
- added link left_ring_DP, mass 0.003002; collision mesh filename=left_sharpa_meshes/left_DP.STL; visual mesh filename=left_sharpa_meshes/left_DP_visual.STL
- added link left_ring_MCP_VL, mass 1.0E-06; collision mesh filename=left_sharpa_meshes/MCP_VL.STL; visual mesh filename=left_sharpa_meshes/left_MCP_VL_visual.STL
- added link left_ring_MP, mass 0.02509; collision mesh filename=left_sharpa_meshes/left_MP.STL; visual mesh filename=left_sharpa_meshes/left_MP_visual.STL
- added link left_ring_PP, mass 0.04138; collision mesh filename=left_sharpa_meshes/left_PP.STL; visual mesh filename=left_sharpa_meshes/left_PP_visual.STL
- added link left_ring_elastomer, mass 0.00110; collision mesh filename=left_sharpa_meshes/elastomer.STL; visual mesh filename=left_sharpa_meshes/elastomer_surface.STL
- added link left_ring_fingertip, mass 1.0E-06
- added link left_thumb_CMC_VL, mass 1.0E-06; visual mesh filename=left_sharpa_meshes/left_thumb_CMC_VL.STL
- added link left_thumb_DP, mass 0.003886; collision mesh filename=left_sharpa_meshes/left_thumb_DP.STL; visual mesh filename=left_sharpa_meshes/left_thumb_DP_visual.STL
- added link left_thumb_MC, mass 0.116; collision mesh filename=left_sharpa_meshes/left_thumb_MC.STL; visual mesh filename=left_sharpa_meshes/left_thumb_MC_visual.STL
- added link left_thumb_MCP_VL, mass 1.0E-06; visual mesh filename=left_sharpa_meshes/left_thumb_MCP_VL_visual.STL
- added link left_thumb_PP, mass 0.04955; collision mesh filename=left_sharpa_meshes/left_thumb_PP.STL; visual mesh filename=left_sharpa_meshes/left_thumb_PP_visual.STL
- added link left_thumb_elastomer, mass 0.002100; collision mesh filename=left_sharpa_meshes/thumb_elastomer.STL; visual mesh filename=left_sharpa_meshes/thumb_elastomer_surface.STL
- added link left_thumb_fingertip, mass 1.0E-06
Joints:
- removed joint right_index_DIP
- removed joint right_index_MCP_AA
- removed joint right_index_MCP_FE
- removed joint right_index_PIP
- removed joint right_index_elastomer_fix_joint
- removed joint right_index_fingertip_fix_joint
- removed joint right_middle_DIP
- removed joint right_middle_MCP_AA
- removed joint right_middle_MCP_FE
- removed joint right_middle_PIP
- removed joint right_middle_elastomer_fix_joint
- removed joint right_middle_fingertip_fix_joint
- removed joint right_pinky_CMC
- removed joint right_pinky_DIP
- removed joint right_pinky_MCP_AA
- removed joint right_pinky_MCP_FE
- removed joint right_pinky_PIP
- removed joint right_pinky_elastomer_fix_joint
- removed joint right_pinky_fingertip_fix_joint
- removed joint right_ring_DIP
- removed joint right_ring_MCP_AA
- removed joint right_ring_MCP_FE
- removed joint right_ring_PIP
- removed joint right_ring_elastomer_fix_joint
- removed joint right_ring_fingertip_fix_joint
- removed joint right_thumb_CMC_AA
- removed joint right_thumb_CMC_FE
- removed joint right_thumb_IP
- removed joint right_thumb_MCP_AA
- removed joint right_thumb_MCP_FE
- removed joint right_thumb_elastomer_fix_joint
- removed joint right_thumb_fingertip_fix_joint
- added joint left_index_DIP: type revolute, parent left_index_MP, child left_index_DP, origin xyz=0.0315 0 0 rpy=0 0 0, axis 0 0 1, limit lower=0 upper=1.3963 effort=0.189369 velocity=14.66594768
- added joint left_index_MCP_AA: type revolute, parent left_index_MCP_VL, child left_index_PP, origin xyz=0 0 0 rpy=1.5708 0 0, axis 0 0 1, limit lower=-0.3491 upper=0.3491 effort=1.864 velocity=16.07692878
- added joint left_index_MCP_FE: type revolute, parent left_hand_C_MC, child left_index_MCP_VL, origin xyz=0.001 -0.0303 0.0957 rpy=0 -1.5708 -1.5708, axis 0 0 1, limit lower=-0.17453293 upper=1.5708 effort=1.864 velocity=16.07692878
- added joint left_index_PIP: type revolute, parent left_index_PP, child left_index_MP, origin xyz=0.047 0 0 rpy=-1.5708 0 0, axis 0 0 1, limit lower=0 upper=1.7453 effort=0.638 velocity=11.61831603
- added joint left_index_elastomer_fix_joint: type fixed, parent left_index_DP, child left_index_elastomer, origin xyz=0 0 0 rpy=1.5707963267949 -1.5707963267949 0, axis 0 0 0
- added joint left_index_fingertip_fix_joint: type fixed, parent left_index_elastomer, child left_index_fingertip, origin xyz=0 -0.0260092574262508 0 rpy=1.5707963267949 1.5707963267949 0, axis 0 0 0
- added joint left_middle_DIP: type revolute, parent left_middle_MP, child left_middle_DP, origin xyz=0.0315 0 0 rpy=0 0 0, axis 0 0 1, limit lower=0 upper=1.3963 effort=0.189369 velocity=14.66594768
- added joint left_middle_MCP_AA: type revolute, parent left_middle_MCP_VL, child left_middle_PP, origin xyz=0 0 0 rpy=1.5708 0 0, axis 0 0 1, limit lower=-0.3491 upper=0.3491 effort=1.864 velocity=16.07692878
- added joint left_middle_MCP_FE: type revolute, parent left_hand_C_MC, child left_middle_MCP_VL, origin xyz=0 -0.01 0.0987 rpy=0 -1.5708 -1.5708, axis 0 0 1, limit lower=-0.17453293 upper=1.5708 effort=1.864 velocity=16.07692878
- added joint left_middle_PIP: type revolute, parent left_middle_PP, child left_middle_MP, origin xyz=0.047 0 0 rpy=-1.5708 0 0, axis 0 0 1, limit lower=0 upper=1.7453 effort=0.638 velocity=11.61831603
- added joint left_middle_elastomer_fix_joint: type fixed, parent left_middle_DP, child left_middle_elastomer, origin xyz=0 0 0 rpy=1.5707963267949 -1.5707963267949 0, axis 0 0 0
- added joint left_middle_fingertip_fix_joint: type fixed, parent left_middle_elastomer, child left_middle_fingertip, origin xyz=0 -0.0260092574262507 0 rpy=1.5707963267949 1.5707963267949 0, axis 0 0 0
- added joint left_pinky_CMC: type revolute, parent left_hand_C_MC, child left_pinky_MC, origin xyz=0.01136 0.0263 0.0867 rpy=-3.1416 0 3.1416, axis 0 0 1, limit lower=0 upper=0.2618 effort=0.5285 velocity=35.07416159
- added joint left_pinky_DIP: type revolute, parent left_pinky_MP, child left_pinky_DP, origin xyz=0.0315 0 0 rpy=0 0 0, axis 0 0 1, limit lower=0 upper=1.3963 effort=0.189369 velocity=14.66594768
- added joint left_pinky_MCP_AA: type revolute, parent left_pinky_MCP_VL, child left_pinky_PP, origin xyz=0 0 0 rpy=1.5708 0 0, axis 0 0 1, limit lower=-0.3491 upper=0.3491 effort=1.864 velocity=16.07692878
- added joint left_pinky_MCP_FE: type revolute, parent left_pinky_MC, child left_pinky_MCP_VL, origin xyz=0.00836 0.0048 0 rpy=-1.5708 1.5708 0, axis 0 0 1, limit lower=-0.17453293 upper=1.5708 effort=1.864 velocity=16.07692878
- added joint left_pinky_PIP: type revolute, parent left_pinky_PP, child left_pinky_MP, origin xyz=0.047 0 0 rpy=-1.5708 0 0, axis 0 0 1, limit lower=0 upper=1.7453 effort=0.638 velocity=11.61831603
- added joint left_pinky_elastomer_fix_joint: type fixed, parent left_pinky_DP, child left_pinky_elastomer, origin xyz=0 0 0 rpy=1.5707963267949 -1.5707963267949 0, axis 0 0 0
- added joint left_pinky_fingertip_fix_joint: type fixed, parent left_pinky_elastomer, child left_pinky_fingertip, origin xyz=0 -0.0260092574262507 0 rpy=1.5707963267949 1.5707963267949 0, axis 0 0 0
- added joint left_ring_DIP: type revolute, parent left_ring_MP, child left_ring_DP, origin xyz=0.0315 0 0 rpy=0 0 0, axis 0 0 1, limit lower=0 upper=1.3963 effort=0.189369 velocity=14.66594768
- added joint left_ring_MCP_AA: type revolute, parent left_ring_MCP_VL, child left_ring_PP, origin xyz=0 0 0 rpy=1.5708 0 0, axis 0 0 1, limit lower=-0.3491 upper=0.3491 effort=1.864 velocity=16.07692878
- added joint left_ring_MCP_FE: type revolute, parent left_hand_C_MC, child left_ring_MCP_VL, origin xyz=0.0015 0.0103 0.0927 rpy=0 -1.5708 -1.5708, axis 0 0 1, limit lower=-0.17453293 upper=1.5708 effort=1.864 velocity=16.07692878
- added joint left_ring_PIP: type revolute, parent left_ring_PP, child left_ring_MP, origin xyz=0.047 0 0 rpy=-1.5708 0 0, axis 0 0 1, limit lower=0 upper=1.7453 effort=0.638 velocity=11.61831603
- added joint left_ring_elastomer_fix_joint: type fixed, parent left_ring_DP, child left_ring_elastomer, origin xyz=0 0 0 rpy=1.5708 -1.5708 0, axis 0 0 0
- added joint left_ring_fingertip_fix_joint: type fixed, parent left_ring_elastomer, child left_ring_fingertip, origin xyz=0 -0.0260092574262507 0 rpy=1.5707963267949 1.5707963267949 0, axis 0 0 0
- added joint left_thumb_CMC_AA: type revolute, parent left_thumb_CMC_VL, child left_thumb_MC, origin xyz=0 -0.005 0 rpy=1.5708 -0.7854 0, axis 0 0 1, limit lower=-0.3491 upper=0.3491 effort=3.3 velocity=11.84076833
- added joint left_thumb_CMC_FE: type revolute, parent left_hand_C_MC, child left_thumb_CMC_VL, origin xyz=0.01 -0.026 0.0212 rpy=0 0 -1.5708, axis 0 0 1, limit lower=-0.1745 upper=1.9199 effort=3.3 velocity=11.84076833
- added joint left_thumb_IP: type revolute, parent left_thumb_PP, child left_thumb_DP, origin xyz=0.039 0 0 rpy=-1.5708 0 0, axis 0 0 1, limit lower=0 upper=1.7453 effort=0.638 velocity=11.61831603
- added joint left_thumb_MCP_AA: type revolute, parent left_thumb_MCP_VL, child left_thumb_PP, origin xyz=0 0 0 rpy=1.5708 0 0, axis 0 0 1, limit lower=-0.3491 upper=0.3491 effort=1.864 velocity=16.07692878
- added joint left_thumb_MCP_FE: type revolute, parent left_thumb_MC, child left_thumb_MCP_VL, origin xyz=0.065 -0.006 -0.010392 rpy=-0.5236 0 0, axis 0 0 1, limit lower=-0.5236 upper=1.3963 effort=1.864 velocity=16.07692878
- added joint left_thumb_elastomer_fix_joint: type fixed, parent left_thumb_DP, child left_thumb_elastomer, origin xyz=0 0 0 rpy=1.5707963267949 -1.5707963267949 0, axis 0 0 0
- added joint left_thumb_fingertip_fix_joint: type fixed, parent left_thumb_elastomer, child left_thumb_fingertip, origin xyz=0 -0.0276109346321216 0 rpy=1.5707963267949 1.5707963267949 0, axis 0 0 0
- joint allegro_mount_joint: child right_hand_C_MC -> left_hand_C_MC
