Commit message: Add adjusted sharpa urdf

File: assets/urdf/kuka_allegro_description/iiwa14_left_sharpa_adjusted.urdf (robot description, URDF)
Before this commit: robot kuka_allegro, 43 links, 42 joints
Links:
- link allegro_mount: geometry collision mesh filename=sharpa_mount.stl scale=0.001 0.001 0.001; visual mesh filename=sharpa_mount.stl scale=0.001 0.001 0.001
Joints:
- joint allegro_mount_joint: origin xyz=0.0 0.0 0.04 rpy=0 0 -1.5708 -> xyz=0.0 0.0 0.05 rpy=0 0 -1.5708

Commit message: Update iiwa14_left_sharpa_adjusted.urdf to use the modified thumb stl and remove mount from geometry

File: assets/urdf/kuka_allegro_description/iiwa14_left_sharpa_adjusted.urdf (robot description, URDF)
Before this commit: robot kuka_allegro, 43 links, 42 joints
Links:
- link allegro_mount: geometry 
- link left_thumb_MC: geometry collision mesh filename=left_sharpa_meshes/left_thumb_MC_modified.STL; visual mesh filename=left_sharpa_meshes/left_thumb_MC_visual.STL

Commit message: Stop using modified thumb

File: assets/urdf/kuka_allegro_description/iiwa14_left_sharpa_adjusted.urdf (robot description, URDF)
Before this commit: robot kuka_allegro, 43 links, 42 joints
Links:
- link left_thumb_MC: geometry collision mesh filename=left_sharpa_meshes/left_thumb_MC.STL; visual mesh filename=left_sharpa_meshes/left_thumb_MC_visual.STL

File: assets/urdf/kuka_allegro_description/iiwa14_left_sharpa_adjusted_restricted.urdf (robot description, URDF)
Before this commit: robot kuka_allegro, 43 links, 42 joints
Links:
- link left_thumb_MC: geometry collision mesh filename=left_sharpa_meshes/left_thumb_MC.STL; visual mesh filename=left_sharpa_meshes/left_thumb_MC_visual.STL
