Commit message: Fix up many things

File: assets/urdf/kuka_allegro_description/iiwa14_real.urdf (robot description, URDF)
Before this commit: robot kuka_allegro, 31 links, 30 joints
Links:
- link allegro_mount: geometry collision mesh filename=meshes/mounts/allegro_mount.obj; visual mesh filename=new_allegro_meshes/mount.stl scale=0.001 0.001 0.001
- link index_link_0: geometry collision mesh filename=meshes/allegro/primary_base.obj; visual mesh filename=meshes/allegro/primary_base.obj
- link index_link_1: geometry collision mesh filename=meshes/allegro/primary_proximal.obj; visual mesh filename=meshes/allegro/primary_proximal.obj
- link index_link_2: geometry collision mesh filename=meshes/allegro/primary_medial.obj; visual mesh filename=meshes/allegro/primary_medial.obj
- link middle_link_0: geometry collision mesh filename=meshes/allegro/primary_base.obj; visual mesh filename=meshes/allegro/primary_base.obj
- link middle_link_1: geometry collision mesh filename=meshes/allegro/primary_proximal.obj; visual mesh filename=meshes/allegro/primary_proximal.obj
- link middle_link_2: geometry collision mesh filename=meshes/allegro/primary_medial.obj; visual mesh filename=meshes/allegro/primary_medial.obj
- link palm_link: geometry collision mesh filename=meshes/allegro/base_link.obj; visual mesh filename=meshes/allegro/base_link.obj
- link ring_link_0: geometry collision mesh filename=meshes/allegro/primary_base.obj; visual mesh filename=meshes/allegro/primary_base.obj
- link ring_link_1: geometry collision mesh filename=meshes/allegro/primary_proximal.obj; visual mesh filename=meshes/allegro/primary_proximal.obj
- link ring_link_2: geometry collision mesh filename=meshes/allegro/primary_medial.obj; visual mesh filename=meshes/allegro/primary_medial.obj
- link thumb_link_0: geometry collision mesh filename=meshes/allegro/thumb_base.obj; visual mesh filename=meshes/allegro/thumb_base.obj
- link thumb_link_1: geometry collision mesh filename=meshes/allegro/thumb_proximal.obj; visual mesh filename=meshes/allegro/thumb_proximal.obj
- link thumb_link_2: geometry collision mesh filename=meshes/allegro/thumb_medial.obj; visual mesh filename=meshes/allegro/thumb_medial.obj

Commit message: Update iiwa14_real mass inertia

File: assets/urdf/kuka_allegro_description/iiwa14_real.urdf (robot description, URDF)
Before this commit: robot kuka_allegro, 31 links, 30 joints
Links:
- link iiwa14_link_1: mass 4 -> 5.76
- link iiwa14_link_2: mass 4 -> 6.35
- link iiwa14_link_3: mass 3 -> 3.50
- link iiwa14_link_4: mass 2.7 -> 3.50
- link iiwa14_link_5: mass 1.7 -> 3.50
- link iiwa14_link_6: mass 1.8 -> 1.80
- link iiwa14_link_7: mass 0.3 -> 1.20
