Commit message: Copy over changes to other urdfs

File: assets/urdf/kuka_allegro_description/iiwa14_h2s2r.urdf (robot description, URDF)
Before this commit: robot kuka_allegro, 64 links, 63 joints
Links:
- link iiwa14_link_1: mass 4 -> 5.76
- link iiwa14_link_2: mass 4 -> 6.35
- link iiwa14_link_3: mass 3 -> 3.50
- link iiwa14_link_4: mass 2.7 -> 3.50
- link iiwa14_link_5: mass 1.7 -> 3.50
- link iiwa14_link_6: mass 1.8 -> 1.80
- link iiwa14_link_7: mass 0.3 -> 1.20

File: assets/urdf/kuka_allegro_description/iiwa14_left_sharpa.urdf (robot description, URDF)
Before this commit: robot kuka_allegro, 43 links, 42 joints
Links:
- link iiwa14_link_1: mass 4 -> 5.76
- link iiwa14_link_2: mass 4 -> 6.35
- link iiwa14_link_3: mass 3 -> 3.50
- link iiwa14_link_4: mass 2.7 -> 3.50
- link iiwa14_link_5: mass 1.7 -> 3.50
- link iiwa14_link_6: mass 1.8 -> 1.80
- link iiwa14_link_7: mass 0.3 -> 1.20

File: assets/urdf/kuka_allegro_description/iiwa14_left_sharpa_adjusted.urdf (robot description, URDF)
Before this commit: robot kuka_allegro, 43 links, 42 joints
Links:
- link iiwa14_link_1: mass 4 -> 5.76
- link iiwa14_link_2: mass 4 -> 6.35
- link iiwa14_link_3: mass 3 -> 3.50
- link iiwa14_link_4: mass 2.7 -> 3.50
- link iiwa14_link_5: mass 1.7 -> 3.50
- link iiwa14_link_6: mass 1.8 -> 1.80
- link iiwa14_link_7: mass 0.3 -> 1.20

File: assets/urdf/kuka_allegro_description/iiwa14_left_sharpa_adjusted_restricted.urdf (robot description, URDF)
Before this commit: robot kuka_allegro, 43 links, 42 joints
Links:
- link iiwa14_link_1: mass 4 -> 5.76
- link iiwa14_link_2: mass 4 -> 6.35
- link iiwa14_link_3: mass 3 -> 3.50
- link iiwa14_link_4: mass 2.7 -> 3.50
- link iiwa14_link_5: mass 1.7 -> 3.50
- link iiwa14_link_6: mass 1.8 -> 1.80
- link iiwa14_link_7: mass 0.3 -> 1.20

File: assets/urdf/kuka_allegro_description/iiwa14_left_sharpa_between.urdf (robot description, URDF)
Before this commit: robot kuka_allegro, 43 links, 42 joints
Links:
- link iiwa14_link_1: mass 4 -> 5.76
- link iiwa14_link_2: mass 4 -> 6.35
- link iiwa14_link_3: mass 3 -> 3.50
- link iiwa14_link_4: mass 2.7 -> 3.50
- link iiwa14_link_5: mass 1.7 -> 3.50
- link iiwa14_link_6: mass 1.8 -> 1.80
- link iiwa14_link_7: mass 0.3 -> 1.20

File: assets/urdf/kuka_allegro_description/iiwa14_real_no_collisions.urdf (robot description, URDF)
Before this commit: robot kuka_allegro, 31 links, 30 joints
Links:
- link iiwa14_link_0: geometry collision mesh filename=new_iiwa14_meshes/collision/link_0.stl; visual mesh filename=new_iiwa14_meshes/visual/link_0.stl
- link iiwa14_link_1: mass 4 -> 5.76; geometry collision mesh filename=new_iiwa14_meshes/collision/link_1.stl; visual mesh filename=new_iiwa14_meshes/visual/link_1.stl
- link iiwa14_link_2: mass 4 -> 6.35; geometry collision mesh filename=new_iiwa14_meshes/collision/link_2.stl; visual mesh filename=new_iiwa14_meshes/visual/link_2.stl
- link iiwa14_link_3: mass 3 -> 3.50; geometry collision mesh filename=new_iiwa14_meshes/collision/link_3.stl; visual mesh filename=new_iiwa14_meshes/visual/link_3.stl
- link iiwa14_link_4: mass 2.7 -> 3.50; geometry collision mesh filename=new_iiwa14_meshes/collision/link_4.stl; visual mesh filename=new_iiwa14_meshes/visual/link_4.stl
- link iiwa14_link_5: mass 1.7 -> 3.50; geometry collision mesh filename=new_iiwa14_meshes/collision/link_5.stl; visual mesh filename=new_iiwa14_meshes/visual/link_5.stl
- link iiwa14_link_6: mass 1.8 -> 1.80; geometry collision mesh filename=new_iiwa14_meshes/collision/link_6.stl; visual mesh filename=new_iiwa14_meshes/visual/link_6.stl
- link iiwa14_link_7: mass 0.3 -> 1.20; geometry collision mesh filename=new_iiwa14_meshes/collision/link_7.stl; visual mesh filename=new_iiwa14_meshes/visual/link_7.stl

File: assets/urdf/kuka_allegro_description/iiwa14_right_sharpa.urdf (robot description, URDF)
Before this commit: robot kuka_allegro, 43 links, 42 joints
Links:
- link iiwa14_link_1: mass 4 -> 5.76
- link iiwa14_link_2: mass 4 -> 6.35
- link iiwa14_link_3: mass 3 -> 3.50
- link iiwa14_link_4: mass 2.7 -> 3.50
- link iiwa14_link_5: mass 1.7 -> 3.50
- link iiwa14_link_6: mass 1.8 -> 1.80
- link iiwa14_link_7: mass 0.3 -> 1.20
