Commit message: Modify mesh filepaths to remove package://

File: assets/urdf/left_sharpa_ha4/left_sharpa_ha4_v2_1.urdf (robot description, URDF)
Before this commit: robot Left_Sharpa_HA4, 33 links, 32 joints
Links:
- link left_hand_C_MC: geometry collision mesh filename=meshes/left_hand_C_MC.STL; visual mesh filename=meshes/left_hand_C_MC_visual.STL
- link left_index_DP: geometry collision mesh filename=meshes/left_DP.STL; visual mesh filename=meshes/left_DP_visual.STL
- link left_index_MCP_VL: geometry collision mesh filename=meshes/MCP_VL.STL; visual mesh filename=meshes/left_MCP_VL_visual.STL
- link left_index_MP: geometry collision mesh filename=meshes/left_MP.STL; visual mesh filename=meshes/left_MP_visual.STL
- link left_index_PP: geometry collision mesh filename=meshes/left_PP.STL; visual mesh filename=meshes/left_PP_visual.STL
- link left_index_elastomer: geometry collision mesh filename=meshes/elastomer.STL; visual mesh filename=meshes/elastomer_surface.STL
- link left_middle_DP: geometry collision mesh filename=meshes/left_DP.STL; visual mesh filename=meshes/left_DP_visual.STL
- link left_middle_MCP_VL: geometry collision mesh filename=meshes/MCP_VL.STL; visual mesh filename=meshes/left_MCP_VL_visual.STL
- link left_middle_MP: geometry collision mesh filename=meshes/left_MP.STL; visual mesh filename=meshes/left_MP_visual.STL
- link left_middle_PP: geometry collision mesh filename=meshes/left_PP.STL; visual mesh filename=meshes/left_PP_visual.STL
- link left_middle_elastomer: geometry collision mesh filename=meshes/elastomer.STL; visual mesh filename=meshes/elastomer_surface.STL
- link left_pinky_DP: geometry collision mesh filename=meshes/left_DP.STL; visual mesh filename=meshes/left_DP_visual.STL
- link left_pinky_MC: geometry collision mesh filename=meshes/left_pinky_MC.STL; visual mesh filename=meshes/left_pinky_MC_visual.STL
- link left_pinky_MCP_VL: geometry collision mesh filename=meshes/MCP_VL.STL; visual mesh filename=meshes/left_MCP_VL_visual.STL
- link left_pinky_MP: geometry collision mesh filename=meshes/left_MP.STL; visual mesh filename=meshes/left_MP_visual.STL
- link left_pinky_PP: geometry collision mesh filename=meshes/left_PP.STL; visual mesh filename=meshes/left_PP_visual.STL
- link left_pinky_elastomer: geometry collision mesh filename=meshes/elastomer.STL; visual mesh filename=meshes/elastomer_surface.STL
- link left_ring_DP: geometry collision mesh filename=meshes/left_DP.STL; visual mesh filename=meshes/left_DP_visual.STL
- link left_ring_MCP_VL: geometry collision mesh filename=meshes/MCP_VL.STL; visual mesh filename=meshes/left_MCP_VL_visual.STL
- link left_ring_MP: geometry collision mesh filename=meshes/left_MP.STL; visual mesh filename=meshes/left_MP_visual.STL
- link left_ring_PP: geometry collision mesh filename=meshes/left_PP.STL; visual mesh filename=meshes/left_PP_visual.STL
- link left_ring_elastomer: geometry collision mesh filename=meshes/elastomer.STL; visual mesh filename=meshes/elastomer_surface.STL
- link left_thumb_CMC_VL: geometry visual mesh filename=meshes/left_thumb_CMC_VL.STL
- link left_thumb_DP: geometry collision mesh filename=meshes/left_thumb_DP.STL; visual mesh filename=meshes/left_thumb_DP_visual.STL
- link left_thumb_MC: geometry collision mesh filename=meshes/left_thumb_MC.STL; visual mesh filename=meshes/left_thumb_MC_visual.STL
- link left_thumb_MCP_VL: geometry visual mesh filename=meshes/left_thumb_MCP_VL_visual.STL
- link left_thumb_PP: geometry collision mesh filename=meshes/left_thumb_PP.STL; visual mesh filename=meshes/left_thumb_PP_visual.STL
- link left_thumb_elastomer: geometry collision mesh filename=meshes/thumb_elastomer.STL; visual mesh filename=meshes/thumb_elastomer_surface.STL

File: assets/urdf/right_sharpa_ha4/right_sharpa_ha4_v2_1.urdf (robot description, URDF)
Before this commit: robot Right_Sharpa_HA4, 33 links, 32 joints
Links:
- link right_hand_C_MC: geometry collision mesh filename=meshes/right_hand_C_MC.STL; visual mesh filename=meshes/right_hand_C_MC_visual.STL
- link right_index_DP: geometry collision mesh filename=meshes/right_DP.STL; visual mesh filename=meshes/right_DP_visual.STL
- link right_index_MCP_VL: geometry collision mesh filename=meshes/MCP_VL.STL; visual mesh filename=meshes/right_MCP_VL_visual.STL
- link right_index_MP: geometry collision mesh filename=meshes/right_MP.STL; visual mesh filename=meshes/right_MP_visual.STL
- link right_index_PP: geometry collision mesh filename=meshes/right_PP.STL; visual mesh filename=meshes/right_PP_visual.STL
- link right_index_elastomer: geometry collision mesh filename=meshes/elastomer.STL; visual mesh filename=meshes/elastomer_surface.STL
- link right_middle_DP: geometry collision mesh filename=meshes/right_DP.STL; visual mesh filename=meshes/right_DP_visual.STL
- link right_middle_MCP_VL: geometry collision mesh filename=meshes/MCP_VL.STL; visual mesh filename=meshes/right_MCP_VL_visual.STL
- link right_middle_MP: geometry collision mesh filename=meshes/right_MP.STL; visual mesh filename=meshes/right_MP_visual.STL
- link right_middle_PP: geometry collision mesh filename=meshes/right_PP.STL; visual mesh filename=meshes/right_PP_visual.STL
- link right_middle_elastomer: geometry collision mesh filename=meshes/elastomer.STL; visual mesh filename=meshes/elastomer_surface.STL
- link right_pinky_DP: geometry collision mesh filename=meshes/right_DP.STL; visual mesh filename=meshes/right_DP_visual.STL
- link right_pinky_MC: geometry collision mesh filename=meshes/right_pinky_MC.STL; visual mesh filename=meshes/right_pinky_MC_visual.STL
- link right_pinky_MCP_VL: geometry collision mesh filename=meshes/MCP_VL.STL; visual mesh filename=meshes/right_MCP_VL_visual.STL
- link right_pinky_MP: geometry collision mesh filename=meshes/right_MP.STL; visual mesh filename=meshes/right_MP_visual.STL
- link right_pinky_PP: geometry collision mesh filename=meshes/right_PP.STL; visual mesh filename=meshes/right_PP_visual.STL
- link right_pinky_elastomer: geometry collision mesh filename=meshes/elastomer.STL; visual mesh filename=meshes/elastomer_surface.STL
- link right_ring_DP: geometry collision mesh filename=meshes/right_DP.STL; visual mesh filename=meshes/right_DP_visual.STL
- link right_ring_MCP_VL: geometry collision mesh filename=meshes/MCP_VL.STL; visual mesh filename=meshes/right_MCP_VL_visual.STL
- link right_ring_MP: geometry collision mesh filename=meshes/right_MP.STL; visual mesh filename=meshes/right_MP_visual.STL
- link right_ring_PP: geometry collision mesh filename=meshes/right_PP.STL; visual mesh filename=meshes/right_PP_visual.STL
- link right_ring_elastomer: geometry collision mesh filename=meshes/elastomer.STL; visual mesh filename=meshes/elastomer_surface.STL
- link right_thumb_CMC_VL: geometry visual mesh filename=meshes/right_thumb_CMC_VL_visual.STL
- link right_thumb_DP: geometry collision mesh filename=meshes/right_thumb_DP.STL; visual mesh filename=meshes/right_thumb_DP_visual.STL
- link right_thumb_MC: geometry collision mesh filename=meshes/right_thumb_MC.STL; visual mesh filename=meshes/right_thumb_MC_visual.STL
- link right_thumb_MCP_VL: geometry visual mesh filename=meshes/right_thumb_MCP_VL_visual.STL
- link right_thumb_PP: geometry collision mesh filename=meshes/right_thumb_PP.STL; visual mesh filename=meshes/right_thumb_PP_visual.STL
- link right_thumb_elastomer: geometry collision mesh filename=meshes/thumb_elastomer.STL; visual mesh filename=meshes/thumb_elastomer_surface.STL
