Commit message: Add assets from main

File: assets/urdf/tyler_objects/blue_cuboid/blue_cuboid.urdf (robot description, URDF)
Before this commit: robot model.urdf, 1 links, 0 joints
Links:
- link baseLink: mass 0.253 -> 0.104; geometry collision mesh filename=cuboid.obj scale=1 1 1; visual mesh filename=cuboid.obj scale=1 1 1

File: assets/urdf/tyler_objects_convex_decomp/hammer_2_2pieces/hammer_2.urdf (robot description, URDF)
Before this commit: robot model.urdf, 1 links, 0 joints
Links:
- link baseLink: geometry collision mesh filename=decomp_0.obj scale=1 1 1; collision mesh filename=decomp_1.obj scale=1 1 1

Commit message: Use cube rotated for clue cuboid

File: assets/urdf/tyler_objects/blue_cuboid/blue_cuboid.urdf (robot description, URDF)
Before this commit: robot model.urdf, 1 links, 0 joints
Links:
- link baseLink: mass 0.104 -> None; geometry collision mesh filename=cuboid_rotated.obj scale=1 1 1; visual mesh filename=cuboid_rotated.obj scale=1 1 1
