Commit message: Do testing on eval_scripts and fix up some objects like spatula

File: assets/urdf/dex_tool_bench/hammer/mallet/mallet.urdf (robot description, URDF)
Before this commit: robot model.urdf, 1 links, 0 joints
Links:
- link baseLink: geometry collision mesh filename=../../../tyler_objects_convex_decomp/mallet/decomp_0.obj scale=1 1 1; collision mesh filename=../../../tyler_objects_convex_decomp/mallet/decomp_1.obj scale=1 1 1

File: assets/urdf/dex_tool_bench/spatula/black_spatula/spatula.urdf (robot description, URDF)
Before this commit: robot spatula, 1 links, 0 joints
Links:
- link spatula: geometry collision mesh filename=../../../tyler_objects_convex_decomp/black_spatula/decomp_0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 scale=1.0 1.0 1.0; collision mesh filename=../../../tyler_objects_convex_decomp/black_spatula/decomp_1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 scale=1.0 1.0 1.0
