Commit message: Add red and red-yellow screwdriver

File: assets/urdf/dex_tool_bench/screwdriver/real_flat_screwdriver/real_flat_screwdriver.urdf (robot description, URDF)
Before this commit: robot model.urdf, 1 links, 0 joints
Links:
- link baseLink: geometry collision mesh filename=../../../tyler_objects_convex_decomp/real_flat_screwdriver/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 scale=1 1 1; collision mesh filename=../../../tyler_objects_convex_decomp/real_flat_screwdriver/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 scale=1 1 1
