Commit message: Fix up red brush

File: assets/urdf/dex_tool_bench/brush/red_brush/red_brush.urdf (robot description, URDF)
Before this commit: robot red_brush, 1 links, 0 joints
Links:
- link red_brush: geometry collision mesh filename=coacd/decomp_0.obj scale=1 1 1; collision mesh filename=coacd/decomp_1.obj scale=1 1 1
